File: hardware/schematic/ser4010.kicad_pcb (KiCad board)
At the start: 2 copper layers, 16 x 35 mm, 39 parts, among them J1 Conn_Coaxial, J2 USB_OTG, J3 3V3, J4 VPP, J5 C2CK, J6 C2D, J7 GND, J8 VBUS, U1 Si4010-GT, U2 CP2102N-A01-GQFN20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

Commit message: HW: fix DI Logo orientation
Parts:
- turned REF** to 270 degrees
Changed lines of the file:
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@@
   )
   (module DI_Logo:DI_Logo (layer B.Cu)
-    (at 162.5 81.5 90)
-    (fp_text reference REF** (at 0 -1.9 90) (layer B.SilkS) hide
+    (at 162.5 81.5 270)
+    (fp_text reference REF** (at 0 -1.9 270) (layer B.SilkS) hide
       (effects (font (size 1 1) (thickness 0.15)) (justify mirror))
     )
-    (fp_text value DI_Logo (at 0 2.025 90) (layer B.Fab) hide
+    (fp_text value DI_Logo (at 0 2.025 270) (layer B.Fab) hide
       (effects (font (size 1 1) (thickness 0.15)) (justify mirror))
     )

Commit message: HW: fix project number
Other:
- board text added: "PN: 0005-00-00"
- board text removed: "PN: 0004-00-00"
Changed lines of the file:
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@@
     (company "Copyright (c) 2018, David Imhoff <dimhoff.devel@gmail.com>")
     (comment 1 "License: BSD-3-Clause")
+    (comment 2 "Project: 0005")
   )
   (layers
@@
     (effects (font (size 0.8 0.8) (thickness 0.15)) (justify mirror))
   )
-  (gr_text "PN: 0004-00-00" (at 162 102.5 90) (layer B.SilkS)
+  (gr_text "PN: 0005-00-00" (at 162 102.5 90) (layer B.SilkS)
     (effects (font (size 0.8 0.8) (thickness 0.15)) (justify mirror))
   )
