File: hardware/schematic/ser4010.sch (KiCad schematic (older format))
At the start: 38 parts, among them J1 Conn_Coaxial, J2 USB_OTG, J3 3V3, J4 VPP, J5 C2CK, J6 C2D, J7 GND, J8 VBUS, U1 Si4010-GT, U2 CP2102N-A01-GQFN20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

Commit message: HW: add part information
Parts:
- C1: Manufacturer (none) -> Murata; Mfr. No (none) -> GRM1555C1H271JA01J; Mouser No (none) -> 81-GRM1555C1H271JA1J; Requirements (none) -> ±5%; C0G (based on 4010-DKPB434-BM_BOM.xls)
- C10: Manufacturer (none) -> Murata; Mfr. No (none) -> GCM1555C1H5R0FA16D; Mouser No (none) -> 81-GCM1555C1H5R0FA6D
- C11, C13: Manufacturer (none) -> Murata; Mfr. No (none) -> GRJ188C70J475KE11D; Mouser No (none) -> 81-GRJ188C70J475KE1D
- C12, C14: Manufacturer (none) -> Wurth Electronics; Mfr. No (none) -> 885012206020; Mouser No (none) -> 710-885012206020
- C2, C4: Manufacturer (none) -> Murata; Mfr. No (none) -> GRM1555C1E6R8BA01D; Mouser No (none) -> 81-GRM1555C1E6R8BA1D; Requirements (none) -> ±5%; C0G (based on 4010-DKPB434-BM_BOM.xls)
- C3: Manufacturer (none) -> Murata; Mfr. No (none) -> GRM1555C1E4R3BA01D; Mouser No (none) -> 81-GRM1555C1E4R3BA1D; Requirements (none) -> ±5%; C0G (based on 4010-DKPB434-BM_BOM.xls)
- C5: Manufacturer (none) -> Murata; Mfr. No (none) -> GRM1555C1H2R7BA01D; Mouser No (none) -> 81-GRM1555C1H2R7BA1D; Requirements (none) -> ±5%; C0G (based on 4010-DKPB434-BM_BOM.xls)
- C6: Manufacturer (none) -> Murata; Mfr. No (none) -> GRM1555C1H1R8WA01D; Mouser No (none) -> 81-GRM1555C1H1R8WA1D; Requirements (none) -> ±5%; C0G (based on 4010-DKPB434-BM_BOM.xls)
- C7: Manufacturer (none) -> Wurth Electronics; Mfr. No (none) -> 885012106018; Mouser No (none) -> 710-885012106018
- C8: Manufacturer (none) -> Murata; Mfr. No (none) -> GRM1555C1H102JA01D; Mouser No (none) -> 81-GRM1555C1H102JA1D
- C9: Manufacturer (none) -> Murata; Mfr. No (none) -> GRM1555C1H271JA01J; Mouser No (none) -> 81-GRM1555C1H271JA1J
- D1: Manufacturer (none) -> Littelfuse; Mfr. No (none) -> SP0503BAHTG; Mouser No (none) -> 576-SP0503BAHTG
- D2: Manufacturer (none) -> Wurth Electronics; Mfr. No (none) -> 150080RS75000; Mouser No (none) -> 710-150080RS75000
- J1: Manufacturer (none) -> Ada Fruit; Mfr. No (none) -> 1865; Mouser No (none) -> 485-1865
- J2: Manufacturer (none) -> FCI / Amphenol; Mfr. No (none) -> 10118193-0001LF; Mouser No (none) -> 649-10118193-0001LF
- J3, J4, J5, J6, J7, J8: Manufacturer (none) -> -; Mfr. No (none) -> -; Mouser No (none) -> -
- L1: Manufacturer (none) -> Coilcraft; Mfr. No (none) -> 0402HP-18NXJLU; Mouser No (none) -> 994-0402HP-18NXJLU; Requirements (none) -> See 'Inductor Selection' sheet
- L2: Manufacturer (none) -> Coilcraft; Mfr. No (none) -> 0402HPH-56NXJLU; Mouser No (none) -> 994-0402HPH-56NXJLU; Requirements (none) -> See 'Inductor Selection' sheet
- L3, L4: Manufacturer (none) -> Coilcraft; Mfr. No (none) -> 0402HP-16NXJLU; Mouser No (none) -> 994-0402HP-16NXJLU; Requirements (none) -> See 'Inductor Selection' sheet
- L5: Manufacturer (none) -> Coilcraft; Mfr. No (none) -> 0402HPH-R22XJLU; Mouser No (none) -> 994-0402HPH-R22XJLU; Requirements (none) -> See 'Inductor Selection' sheet
- U1: Manufacturer (none) -> Silicon Laboratories; Mfr. No (none) -> SI4010-C2-GT; Mouser No (none) -> 634-SI4010-C2-GT
- U2: Manufacturer (none) -> Silicon Laboratories; Mfr. No (none) -> CP2102NA01GQFN20; Mouser No (none) -> 634-CP2102NA01GQFN20
- Y1: Manufacturer (none) -> IQD Frequency Products; Mfr. No (none) -> LFXTAL055915; Mouser No (none) -> 449-LFXTAL055915REEL
